Commit message: Project 1 - completed without exercise 8, because the PD regulator implementation is described in later steps

File: urdf/planar2dof.urdf (robot description, URDF)
Before this commit: robot planar2dof, 5 links, 4 joints
Links:
- link planar2dof/link_striker_ee: mass 0.1 -> 3

Commit message: Completed mini-projects 1 and 2. Not yet confirmed if the recieved parameters are correct. Will ask.

File: urdf/planar2dof.urdf (robot description, URDF)
Before this commit: robot planar2dof, 5 links, 4 joints
Links:
- link planar2dof/link_striker_ee: mass 3 -> 0.1
